File: mpt_sleep_control.kicad_sch (KiCad schematic)
At the start: 6 parts, among them SW1 OS102011MA1QN1

Commit message: Make Block Titles consistent in size Remove not connected marks on mcu for pins which can be used for user buttons and other stuff Add User button hierarchy lables for Button 4 & 5 on MCU sheet Fix hierarchichal pin names on the block not matching the sheet
Parts:
- R1, R2, R4: now not fitted
Other:
- title: (none) -> M.P.T. Sleep Control
Changed lines of the file:
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@@
 	(paper "A4")
 	(title_block
+		(title "M.P.T. Sleep Control")
 		(company "Hochschule Luzern, Technik & Architektur")
+		(comment 1 "Designed by Nico Theiler & Dominik Grob")
 	)
 	(text "Buck Shutdown:\nThe Buckconverter is shutdown. Only the BMS and \nthe RTC get power from the batteries.\nMCU Shutdown:\nThe MCU get the signal to shutdown and goes into deepsleep."
@@
 		(on_board yes)
 		(in_pos_files yes)
-		(dnp no)
+		(dnp yes)
 		(property "Reference" "R4"
 			(at 168.656 69.9657 0)
@@
 		(on_board yes)
 		(in_pos_files yes)
-		(dnp no)
+		(dnp yes)
 		(property "Reference" "R1"
 			(at 126.746 100.4457 0)
@@
 		(on_board yes)
 		(in_pos_files yes)
-		(dnp no)
+		(dnp yes)
 		(fields_autoplaced yes)
 		(property "Reference" "R2"
