File: MPT.kicad_pcb (KiCad board)
At the start: 2 copper layers, 60 x 50 mm, 94 parts, among them J1 USB4105GFA120, J2 ER-TFT2.79-1, Q2 BSS138, SW1 OS102011MA1QN1, SW2 KMR421GULCLFS, SW3 KMR421GULCLFS, SW4 SW_1825910-6, SW5 SW_1825910-6, SW6 SW_1825910-6, SW7 SW_1825910-6, U2 BQ25185, U3 BQ27441-G1, U4 ESP32-S3-WROOM-1-N4R2, U5 RCLAMP0854P.TCT, U6 TPS63030, U7 MIC2841A

Commit message: Final Changes 1
Routing:
- net SHELL_GND: track 18.9 -> 19.5 mm
- net GND: vias 221 -> 224
- net +3V4: vias 36 -> 34
Changed lines of the file:
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@@
 		(tags "resistor")
 		(property "Reference" "R12"
-			(at 2.5 0 90)
+			(at 2.55 -0.25 90)
 			(layer "F.SilkS")
 			(effects
@@
 		(at 176.553602 119.961009 -135)
 		(property "Reference" "S1"
-			(at -5.515433 3.535534 0)
+			(at -5.374012 2.616295 0)
 			(layer "B.SilkS")
 			(effects
@@
 	)
 	(via
+		(at 159.503602 130.711009)
+		(size 0.6)
+		(drill 0.3)
+		(layers "F.Cu" "B.Cu")
+		(free yes)
+		(net "GND")
+	)
+	(via
 		(at 166.653602 120.661009)
 		(size 0.6)
@@
 	)
 	(via
+		(at 164.103602 130.711009)
+		(size 0.6)
+		(drill 0.3)
+		(layers "F.Cu" "B.Cu")
+		(free yes)
+		(net "GND")
+	)
+	(via
 		(at 140.603602 104.111009)
 		(size 0.6)
@@
 	)
 	(via
+		(at 161.803602 130.761009)
+		(size 0.6)
+		(drill 0.3)
+		(layers "F.Cu" "B.Cu")
+		(free yes)
+		(net "GND")
+	)
+	(via
 		(at 129.203602 92.561009)
 		(size 0.6)
@@
 	)
 	(via
-		(at 138.019102 101.895509)
-		(size 0.6)
-		(drill 0.3)
-		(layers "F.Cu" "B.Cu")
-		(net "+3V4")
-	)
-	(via
 		(at 173.053602 98.961009)
 		(size 0.6)
@@
 	)
 	(via
-		(at 135.553602 115.061009)
-		(size 0.6)
-		(drill 0.3)
-		(layers "F.Cu" "B.Cu")
-		(net "+3V4")
-	)
-	(via
 		(at 181.453602 116.661009)
 		(size 0.6)
@@
 	)
 	(segment
+		(start 166.2185 130.7526)
+		(end 165.460091 131.511009)
+		(width 0.4)
+		(layer "B.Cu")
+		(net "SHELL_GND")
+	)
+	(segment
 		(start 157.5785 126.5726)
 		(end 157.5785 130.7526)
@@
 	)
 	(segment
-		(start 166.2185 130.7526)
+		(start 165.460091 131.511009)
+		(end 158.336909 131.511009)
+		(width 0.4)
+		(layer "B.Cu")
+		(net "SHELL_GND")
+	)
+	(segment
+		(start 158.336909 131.511009)
 		(end 157.5785 130.7526)
 		(width 0.4)
@@
 		)
 		(min_thickness 0.25)
-		(fill yes
+		(fill
 			(thermal_gap 0.5)
 			(thermal_bridge_width 0.5)
@@
 		(polygon
 			(pts
-				(xy 109.703602 75.861009) (xy 204.003602 75.511009) (xy 204.603602 138.911009) (xy 109.203602 136.611009)
+				(xy 108.453602 77.011009) (xy 203.303602 76.411009) (xy 202.653602 137.611009) (xy 108.803602 137.661009)
 			)
 		)
